Commit message: fix: motion, visibility, and grid-localisation bugs
Four distinct problems surfaced from the first heartbeat-enabled run:

1. diff_drive plugin was subscribing to relative 'cmd_vel' → got
   namespaced to /model/artpark_bot/cmd_vel under the hood. Our bridge
   talks to /cmd_vel (absolute), so the plugin never received twists.
   Use absolute /cmd_vel and /odom in the URDF plugin tags.

2. <gazebo><material>Gazebo/Grey</material></gazebo> uses a deprecated
   Ogre script path and silently broke rendering on Harmonic. Remove it;
   the URDF-level <material name='body_grey'/> with rgba already covers
   visualisation.

3. tile_tracker was treating odom pose (starts at 0,0 relative to spawn)
   as world pose. Robot spawned at world (-1.35, 1.8) but tile_tracker
   reported tile=(2,1). Add spawn_world_x/y parameters wired through
   full_run.launch.py so the offset is applied before world_to_tile().

4. state_machine._edge_to_yaw used a non-compass convention
   (N → yaw=0) while tile_tracker.edge_crossed treats N = +y
   (compass). Align both on the standard compass:
     N = +y = yaw π/2
     E = +x = yaw 0
     S = -y = yaw -π/2
     W = -x = yaw π

File: src/artpark_robot/urdf/artpark_bot.urdf.xacro (robot description, xacro)
@@ -152,7 +152,6 @@
   </joint>
   <!-- ================= GAZEBO / IGNITION TAGS ================= -->
-  <gazebo reference="base_link">
-    <material>Gazebo/Grey</material>
-  </gazebo>
+  <!-- Friction only; DON'T override material (URDF visuals already set colour
+       and Gazebo/Grey is deprecated — its warning broke rendering for us). -->
   <gazebo reference="wheel_left">
     <mu1>1.0</mu1><mu2>1.0</mu2>
@@ -164,5 +163,7 @@
     <mu1>0.0</mu1><mu2>0.0</mu2>
   </gazebo>
-  <!-- Differential drive plugin -->
+  <!-- Differential drive plugin.
+       Topic names are absolute (leading slash) so they don't get namespaced
+       under /model/artpark_bot/ — the bridge talks to /cmd_vel + /odom. -->
   <gazebo>
     <plugin filename="gz-sim-diff-drive-system"
@@ -172,6 +173,6 @@
       <wheel_separation>${wheel_sep}</wheel_separation>
       <wheel_radius>${wheel_rad}</wheel_radius>
-      <topic>cmd_vel</topic>
-      <odom_topic>odom</odom_topic>
+      <topic>/cmd_vel</topic>
+      <odom_topic>/odom</odom_topic>
       <frame_id>odom</frame_id>
       <child_frame_id>base_footprint</child_frame_id>
@@ -181,5 +182,5 @@
     <plugin filename="gz-sim-joint-state-publisher-system"
             name="gz::sim::systems::JointStatePublisher">
-      <topic>joint_states</topic>
+      <topic>/joint_states</topic>
     </plugin>
   </gazebo>

Commit message: feat: explicit Gazebo materials, debug_hold mode, odom in heartbeat
Visibility:
- Added <gazebo reference='X'><visual><material><ambient/diffuse>...
  for base_link (bright red), wheels (black), cameras (blue), LiDAR
  (yellow). SDF-style materials render reliably on Harmonic; relying on
  URDF-only <material name=...> was inconsistent.

Diagnostics:
- state_machine now carries odom_x / odom_y in its state and prints them
  in the 2 Hz heartbeat line so operators can compare (odom origin +
  spawn_pose) against the reported tile.
- New debug_hold launch arg. When true, the state machine stays in INIT
  forever and never emits cmd_vel. Lets us inspect spawn pose without
  the robot wandering off.

No behaviour change when debug_hold=false (default).

File: src/artpark_robot/urdf/artpark_bot.urdf.xacro (robot description, xacro)
@@ -152,14 +152,51 @@
   </joint>
   <!-- ================= GAZEBO / IGNITION TAGS ================= -->
-  <!-- Friction only; DON'T override material (URDF visuals already set colour
-       and Gazebo/Grey is deprecated — its warning broke rendering for us). -->
+  <!-- Explicit inline materials per link (ambient + diffuse). This is the
+       SDF-native form that Gazebo Harmonic renders reliably; URDF-only
+       <material name=...> blocks are not always picked up by sdformat.
+       Chose deliberately loud colours to make the robot obvious. -->
+  <gazebo reference="base_link">
+    <visual>
+      <material>
+        <ambient>1.0 0.1 0.1 1.0</ambient>
+        <diffuse>1.0 0.1 0.1 1.0</diffuse>
+        <specular>0.2 0.2 0.2 1.0</specular>
+      </material>
+    </visual>
+  </gazebo>
   <gazebo reference="wheel_left">
     <mu1>1.0</mu1><mu2>1.0</mu2>
+    <visual><material>
+      <ambient>0.05 0.05 0.05 1.0</ambient>
+      <diffuse>0.05 0.05 0.05 1.0</diffuse>
+    </material></visual>
   </gazebo>
   <gazebo reference="wheel_right">
     <mu1>1.0</mu1><mu2>1.0</mu2>
+    <visual><material>
+      <ambient>0.05 0.05 0.05 1.0</ambient>
+      <diffuse>0.05 0.05 0.05 1.0</diffuse>
+    </material></visual>
   </gazebo>
   <gazebo reference="caster">
     <mu1>0.0</mu1><mu2>0.0</mu2>
+  </gazebo>
+  <gazebo reference="front_cam">
+    <visual><material>
+      <ambient>0.1 0.3 0.9 1.0</ambient>
+      <diffuse>0.1 0.3 0.9 1.0</diffuse>
+    </material></visual>
+  </gazebo>
+  <gazebo reference="floor_cam">
+    <visual><material>
+      <ambient>0.1 0.3 0.9 1.0</ambient>
+      <diffuse>0.1 0.3 0.9 1.0</diffuse>
+    </material></visual>
+  </gazebo>
+  <gazebo reference="lidar_link">
+    <visual><material>
+      <ambient>1.0 0.8 0.0 1.0</ambient>
+      <diffuse>1.0 0.8 0.0 1.0</diffuse>
+    </material></visual>
   </gazebo>
   <!-- Differential drive plugin.

Commit message: fix: work around argparse negative-value bug in spawn + add fallback teleport
Root cause: at first heartbeat the robot was already at tile (2,2) which
is world (0.45, 0.0) — exactly where Gazebo defaults spawn would land if
our -x/-y args were ignored. The ros_gz_sim/create CLI uses argparse,
which mis-parses '-x -1.35' because the value '-1.35' starts with '-'
and argparse treats it as another flag.

Fix uses three defences:

1. ExecuteProcess instead of Node with argv list form '[-x, =, value]'
   which the launch system joins without a space, producing '-x=-1.35'.
   That's the argparse-safe form for negative values.

2. After-spawn TimerAction calls gz service /world/artpark_arena/set_pose
   with reqtype Pose, reptype Boolean. Belt-and-suspenders teleport to
   the intended world pose in case (1) still drops args.

3. base_footprint now has a minimal inertial block. Some SDF spawn paths
   refuse a root link without inertial properties.

File: src/artpark_robot/urdf/artpark_bot.urdf.xacro (robot description, xacro)
@@ -44,5 +44,12 @@
   </xacro:macro>
   <!-- ================= CHASSIS ================= -->
-  <link name="base_footprint"/>
+  <!-- base_footprint is the root frame. Some spawn tools require an
+       inertial on the root link; give it a tiny non-zero one. -->
+  <link name="base_footprint">
+    <inertial>
+      <mass value="0.001"/>
+      <inertia ixx="1e-6" ixy="0" ixz="0" iyy="1e-6" iyz="0" izz="1e-6"/>
+    </inertial>
+  </link>
   <link name="base_link">
     <xacro:inertial_box mass="${base_mass}" x="${base_len}" y="${base_wid}" z="${base_hei}"/>
